Commit message: navigation is added

File: urdf/mecanum_robot.xacro (robot description, xacro)
@@ -2,43 +2,32 @@
 <robot name="mecanum_robot" xmlns:xacro="http://www.ros.org/wiki/xacro">
   <xacro:include filename="$(find mecanum_robot)/urdf/mecanum_robot.gazebo" />
-<!-- .............Robot Footprint & Chassis................................................... -->
-  <link name="robot_footprint"></link>
-  <link
-    name="chassis">
-    <inertial>
-      <origin
-        xyz="-8.294E-05 -7.7011E-11 -0.023972"
-        rpy="0 0 0" />
-      <mass
-        value="6.5996" />
-      <inertia
-        ixx="0.043356"
-        ixy="-1.6809E-08"
-        ixz="-1.7057E-07"
-        iyy="0.13461"
-        iyz="3.8673E-11"
-        izz="0.17533" />
-    </inertial>
-    <visual>
-      <origin
-        xyz="0 0 0"
-        rpy="0 0 0" />
-      <geometry>
-        <mesh
-          filename="package://mecanum_robot/meshes/chassis.STL" />
-      </geometry>
-      <material
-        name="">
-        <color
-          rgba="0.79216 0.81961 0.93333 1" />
-      </material>
-    </visual>
-    <collision>
-      <origin
-        xyz="0 0 0"
-        rpy="0 0 0" />
-      <geometry>
-        <mesh
-          filename="package://mecanum_robot/meshes/chassis.STL" />
+<!-- .............Robot Footprint & Chassis (Link - Joint).......................................... -->
+  <link name="robot_footprint">
+    <visual>
+      <origin xyz="0 0 0" rpy="0 0 0" />
+      <geometry>
+        <box size="0.001 0.001 0.001" />
+      </geometry>
+    </visual>
+  </link>
+  <link name="chassis">
+    <inertial>
+      <origin xyz="-8.294E-05 -7.7011E-11 -0.023972" rpy="0 0 0" />
+      <mass value="6.5996" />
+      <inertia ixx="0.043356" ixy="-1.6809E-08" ixz="-1.7057E-07" iyy="0.13461" iyz="3.8673E-11" izz="0.17533" />
+    </inertial>
+    <visual>
+      <origin xyz="0 0 0" rpy="0 0 0" />
+      <geometry>
+        <mesh filename="package://mecanum_robot/meshes/chassis.STL" />
+      </geometry>
+      <material name="">
+        <color rgba="0.79216 0.81961 0.93333 1" />
+      </material>
+    </visual>
+    <collision>
+      <origin xyz="0 0 0" rpy="0 0 0" />
+      <geometry>
+        <mesh filename="package://mecanum_robot/meshes/chassis.STL" />
       </geometry>
     </collision>
@@ -49,242 +38,162 @@
     <child link="chassis" />
   </joint>
-<!-- ................Rear Right Wheel................................................ -->
-  <link
-    name="rear_right_wheel">
-    <inertial>
-      <origin
-        xyz="1.624E-12 -3.4926E-12 0.021031"
-        rpy="0 0 0" />
-      <mass
-        value="0.049871" />
-      <inertia
-        ixx="5.3189E-06"
-        ixy="1.2084E-15"
-        ixz="-9.388E-17"
-        iyy="5.3189E-06"
-        iyz="1.994E-16"
-        izz="6.4396E-06" />
-    </inertial>
-    <visual>
-      <origin
-        xyz="0 0 0"
-        rpy="0 0 0" />
-      <geometry>
-        <mesh
-          filename="package://mecanum_robot/meshes/rear_right_wheel.STL" />
-      </geometry>
-      <material
-        name="">
-        <color
-          rgba="0.79216 0.81961 0.93333 1" />
-      </material>
-    </visual>
-    <collision>
-      <origin
-        xyz="0 0 0"
-        rpy="0 0 0" />
-      <geometry>
-        <mesh
-          filename="package://mecanum_robot/meshes/rear_right_wheel.STL" />
-      </geometry>
-    </collision>
-  </link>
-  <joint
-    name="rear_right_wheel_joint"
-    type="continuous">
-    <origin
-      xyz="0.1175 0.113 -0.03"
-      rpy="1.5708 -0.55618 3.1416" />
-    <parent
-      link="chassis" />
-    <child
-      link="rear_right_wheel" />
-    <axis
-      xyz="0 0 1" />
-    <limit
-      lower="-3.14"
-      upper="3.14"
-      effort="200"
-      velocity="5" />
-  </joint>
-<!-- ..................Rear Left Wheel............................................... -->
-  <link
-    name="rear_left_wheel">
-    <inertial>
-      <origin
-        xyz="-6.2922E-13 3.7938E-12 0.021031"
-        rpy="0 0 0" />
-      <mass
-        value="0.049871" />
-      <inertia
-        ixx="5.3189E-06"
-        ixy="5.4099E-16"
-        ixz="3.9906E-17"
-        iyy="5.3189E-06"
-        iyz="-2.1312E-16"
-        izz="6.4396E-06" />
-    </inertial>
-    <visual>
-      <origin
-        xyz="0 0 0"
-        rpy="0 0 0" />
-      <geometry>
-        <mesh
-          filename="package://mecanum_robot/meshes/rear_left_wheel.STL" />
-      </geometry>
-      <material
-        name="">
-        <color
-          rgba="0.79216 0.81961 0.93333 1" />
-      </material>
-    </visual>
-    <collision>
-      <origin
-        xyz="0 0 0"
-        rpy="0 0 0" />
-      <geometry>
-        <mesh
-          filename="package://mecanum_robot/meshes/rear_left_wheel.STL" />
-      </geometry>
-    </collision>
-  </link>
-  <joint
-    name="rear_left_wheel_joint"
-    type="continuous">
-    <origin
-      xyz="0.1175 -0.113 -0.03"
-      rpy="-1.5708 -1.0094 3.1416" />
-    <parent
-      link="chassis" />
-    <child
-      link="rear_left_wheel" />
-    <axis
-      xyz="0 0 1" />
-    <limit
-      lower="-3.14"
-      upper="3.14"
-      effort="200"
-      velocity="5" />
-  </joint>
-<!-- ....................Front Right Wheel..................................................... -->
-  <link
-    name="front_right_wheel">
-    <inertial>
-      <origin
-        xyz="-6.2939E-13 3.7953E-12 0.021031"
-        rpy="0 0 0" />
-      <mass
-        value="0.049871" />
-      <inertia
-        ixx="5.3189E-06"
-        ixy="5.4109E-16"
-        ixz="3.6773E-17"
-        iyy="5.3189E-06"
-        iyz="-2.1556E-16"
-        izz="6.4396E-06" />
-    </inertial>
-    <visual>
-      <origin
-        xyz="0 0 0"
-        rpy="0 0 0" />
-      <geometry>
-        <mesh
-          filename="package://mecanum_robot/meshes/front_right_wheel.STL" />
-      </geometry>
-      <material
-        name="">
-        <color
-          rgba="0.79216 0.81961 0.93333 1" />
-      </material>
-    </visual>
-    <collision>
-      <origin
-        xyz="0 0 0"
-        rpy="0 0 0" />
-      <geometry>
-        <mesh
-          filename="package://mecanum_robot/meshes/front_right_wheel.STL" />
-      </geometry>
-    </collision>
-  </link>
-  <joint
-    name="front_right_wheel_joint"
-    type="continuous">
-    <origin
-      xyz="-0.1175 0.113 -0.03"
-      rpy="1.5708 0.55618 3.1416" />
-    <parent
-      link="chassis" />
-    <child
-      link="front_right_wheel" />
-    <axis
-      xyz="0 0 1" />
-    <limit
-      lower="-3.14"
-      upper="3.14"
-      effort="200"
-      velocity="5" />
-  </joint>
-<!-- ..................Front Left Wheel....................................................... -->
-  <link
-    name="front_left_wheel">
-    <inertial>
-      <origin
-        xyz="1.451E-12 -3.5752E-12 0.021031"
-        rpy="0 0 0" />
-      <mass
-        value="0.049871" />
-      <inertia
-        ixx="5.3189E-06"
-        ixy="1.1259E-15"
-        ixz="-8.0856E-17"
-        iyy="5.3189E-06"
-        iyz="2.0104E-16"
-        izz="6.4396E-06" />
-    </inertial>
-    <visual>
-      <origin
-        xyz="0 0 0"
-        rpy="0 0 0" />
-      <geometry>
-        <mesh
-          filename="package://mecanum_robot/meshes/front_left_wheel.STL" />
-      </geometry>
-      <material
-        name="">
-        <color
-          rgba="0.79216 0.81961 0.93333 1" />
-      </material>
-    </visual>
-    <collision>
-      <origin
-        xyz="0 0 0"
-        rpy="0 0 0" />
-      <geometry>
-        <mesh
-          filename="package://mecanum_robot/meshes/front_left_wheel.STL" />
-      </geometry>
-    </collision>
-  </link>
-  <joint
-    name="front_left_wheel_joint"
-    type="continuous">
-    <origin
-      xyz="-0.1175 -0.113 -0.03"
-      rpy="-1.5708 1.3416 3.1416" />
-    <parent
-      link="chassis" />
-    <child
-      link="front_left_wheel" />
-    <axis
-      xyz="0 0 1" />
-    <limit
-      lower="-3.14"
-      upper="3.14"
-      effort="200"
-      velocity="5" />
-  </joint>
-<!-- ............................Camera........................................... -->
-  <link name="camera">
+<!-- ................Rear Right Wheel (Link - Joint - Transmission)................................ -->
+  <link name="rear_right_wheel">
+    <inertial>
+      <origin xyz="1.624E-12 -3.4926E-12 0.021031" rpy="0 0 0" />
+      <mass value="0.049871" />
+      <inertia ixx="5.3189E-06" ixy="1.2084E-15" ixz="-9.388E-17" iyy="5.3189E-06" iyz="1.994E-16" izz="6.4396E-06" />
+    </inertial>
+    <visual>
+      <origin xyz="0 0 0" rpy="0 0 0" />
+      <geometry>
+        <mesh filename="package://mecanum_robot/meshes/rear_right_wheel.STL" />
+      </geometry>
+      <material name="">
+        <color rgba="0.79216 0.81961 0.93333 1" />
+      </material>
+    </visual>
+    <collision>
+      <origin xyz="0 0 0" rpy="0 0 0" />
+      <geometry>
+        <mesh filename="package://mecanum_robot/meshes/rear_right_wheel.STL" />
+      </geometry>
+    </collision>
+  </link>
+  <joint name="rear_right_wheel_joint" type="continuous">
+    <origin xyz="0.1175 0.113 -0.03" rpy="1.5708 -0.55618 3.1416" />
+    <parent link="chassis" />
+    <child link="rear_right_wheel" />
+    <axis xyz="0 0 1" />
+    <limit lower="-3.14" upper="3.14" effort="200" velocity="5" />
+  </joint>
+  <transmission name="rear_right_wheel_joint_trans">
+    <type>transmission_interface/SimpleTransmission</type>
+    <joint name="rear_right_wheel_joint" >
+      <hardwareInterface>hardware_interface/VelocityJointInterface</hardwareInterface>
+    </joint>
+    <actuator name="rear_right_wheel_joint_motor">
+        <mechanicalReduction>1</mechanicalReduction>
+    </actuator>
+  </transmission>
+<!-- ..................Rear Left Wheel (Link - Joint - Transmission)................................ -->
+  <link name="rear_left_wheel">
+    <inertial>
+      <origin xyz="-6.2922E-13 3.7938E-12 0.021031" rpy="0 0 0" />
+      <mass value="0.049871" />
+      <inertia ixx="5.3189E-06" ixy="5.4099E-16" ixz="3.9906E-17" iyy="5.3189E-06" iyz="-2.1312E-16" izz="6.4396E-06" />
+    </inertial>
+    <visual>
+      <origin xyz="0 0 0" rpy="0 0 0" />
+      <geometry>
+        <mesh filename="package://mecanum_robot/meshes/rear_left_wheel.STL" />
+      </geometry>
+      <material name="">
+        <color rgba="0.79216 0.81961 0.93333 1" />
+      </material>
+    </visual>
+    <collision>
+      <origin xyz="0 0 0" rpy="0 0 0" />
+      <geometry>
+        <mesh filename="package://mecanum_robot/meshes/rear_left_wheel.STL" />
+      </geometry>
+    </collision>
+  </link>
+  <joint name="rear_left_wheel_joint" type="continuous">
+    <origin xyz="0.1175 -0.113 -0.03" rpy="-1.5708 -1.0094 3.1416" />
+    <parent link="chassis" />
+    <child link="rear_left_wheel" />
+    <axis xyz="0 0 1" />
+    <limit lower="-3.14" upper="3.14" effort="200" velocity="5" />
+  </joint>
+  <transmission name="rear_left_wheel_joint_trans">
+    <type>transmission_interface/SimpleTransmission</type>
+    <joint name="rear_left_wheel_joint" >
+      <hardwareInterface>hardware_interface/VelocityJointInterface</hardwareInterface>
+    </joint>
+    <actuator name="rear_left_wheel_joint_motor">
+        <mechanicalReduction>1</mechanicalReduction>
+    </actuator>
+  </transmission>
+<!-- ....................Front Right Wheel (Link - Joint - Transmission)................................ -->
+  <link name="front_right_wheel">
+    <inertial>
+      <origin xyz="-6.2939E-13 3.7953E-12 0.021031" rpy="0 0 0" />
+      <mass value="0.049871" />
+      <inertia ixx="5.3189E-06" ixy="5.4109E-16" ixz="3.6773E-17" iyy="5.3189E-06" iyz="-2.1556E-16" izz="6.4396E-06" />
+    </inertial>
+    <visual>
+      <origin xyz="0 0 0" rpy="0 0 0" />
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
Commit message: navigation update

File: urdf/mecanum_robot.xacro (robot description, xacro)
@@ -1,14 +1,10 @@
 <?xml version='1.0'?>
 <robot name="mecanum_robot" xmlns:xacro="http://www.ros.org/wiki/xacro">
-  <xacro:include filename="$(find mecanum_robot)/urdf/mecanum_robot.gazebo" />
+<xacro:include filename="$(find mecanum_robot)/urdf/mecanum_robot.gazebo" />
+  <!-- Wheels -->
+  <xacro:property name="r" value="0.03" /> <!-- wheel radius in m-->
+  <xacro:property name="h" value="0.03" /> <!-- wheel length in m-->
 <!-- .............Robot Footprint & Chassis (Link - Joint).......................................... -->
-  <link name="robot_footprint">
-    <visual>
-      <origin xyz="0 0 0" rpy="0 0 0" />
-      <geometry>
-        <box size="0.001 0.001 0.001" />
-      </geometry>
-    </visual>
-  </link>
+  <link name="robot_footprint"/>
   <link name="chassis">
     <inertial>
@@ -29,10 +25,10 @@
       <origin xyz="0 0 0" rpy="0 0 0" />
       <geometry>
-        <mesh filename="package://mecanum_robot/meshes/chassis.STL" />
+	      <mesh filename="package://mecanum_robot/meshes/chassis.STL" />
       </geometry>
     </collision>
   </link>
   <joint name="robot_footprint_joint" type="fixed">
-    <origin xyz="0 0 0" rpy="0 0 0" />
+    <origin xyz="0 0 0.05" rpy="0 0 0" />
     <parent link="robot_footprint"/>
     <child link="chassis" />
@@ -57,5 +53,5 @@
       <origin xyz="0 0 0" rpy="0 0 0" />
       <geometry>
-        <mesh filename="package://mecanum_robot/meshes/rear_right_wheel.STL" />
+        <cylinder length="${h}" radius="${r}" />
       </geometry>
     </collision>
@@ -96,5 +92,5 @@
       <origin xyz="0 0 0" rpy="0 0 0" />
       <geometry>
-        <mesh filename="package://mecanum_robot/meshes/rear_left_wheel.STL" />
+        <cylinder length="${h}" radius="${r}" />
       </geometry>
     </collision>
@@ -135,5 +131,5 @@
       <origin xyz="0 0 0" rpy="0 0 0" />
       <geometry>
-        <mesh filename="package://mecanum_robot/meshes/front_right_wheel.STL" />
+        <cylinder length="${h}" radius="${r}" />
       </geometry>
     </collision>
@@ -174,5 +170,5 @@
       <origin xyz="0 0 0" rpy="0 0 0" />
       <geometry>
-        <mesh filename="package://mecanum_robot/meshes/front_left_wheel.STL" />
+        <cylinder length="${h}" radius="${r}" />
       </geometry>
     </collision>
@@ -195,5 +191,5 @@
   </transmission>
 <!-- ............................Camera (Link - Joint)..................................... -->
-  <!-- <link name="camera">
+  <link name="camera">
     <inertial>
       <origin xyz="0 0 0" rpy="0 0 0"/>
@@ -204,11 +200,11 @@
       <origin xyz="0 0 0" rpy="0 0 0"/>
       <geometry>
-        <box size="0.05 0.05 0.05"/>
-      </geometry>
-    </collision>
-    <visual>
-      <origin xyz="0 0 0" rpy="0 0 0"/>
-      <geometry>
-        <box size="0.05 0.05 0.05"/>
+        <box size="0.04 0.04 0.04"/>
+      </geometry>
+    </collision>
+    <visual>
+      <origin xyz="0 0 0" rpy="0 0 0"/>
+      <geometry>
+        <box size="0.04 0.04 0.04"/>
       </geometry>
     </visual>
@@ -219,5 +215,5 @@
     <child link="camera"/>
     <axis xyz="0.0 1.0 0.0"/>
-  </joint> -->
+  </joint>
 <!-- .........................Lidar (Link - Joint)................................... -->
   <link name="hokuyo">
@@ -244,5 +240,5 @@
     <parent link="chassis"/>
     <child link="hokuyo"/>
-    <axis xyz="0.0 1.0 0.0"/>
+    <axis xyz="0.0 1.0 0.2"/>
   </joint>
 </robot>
